Commit message: Add hector_slam and set planner params

File: src/wheelchair_description/urdf/wheelchair_body_stereo.xacro (robot description, xacro)
@@ -7,6 +7,6 @@
   <xacro:property name="base_dia" value="0.5"/>
   <!-- along z axis -->
-  <xacro:property name="base_height" value="0.095"/>
-  <xacro:property name="base_mass" value="15"/>
+  <xacro:property name="base_height" value="0.099"/>
+  <xacro:property name="base_mass" value="50"/>
   <xacro:property name="wheel_dia" value="0.1"/>
   <xacro:property name="wheel_height" value="0.05"/>
@@ -100,100 +100,27 @@
   <xacro:wheel left_right="left" rely="1"/>
   <xacro:wheel left_right="right" rely="-1"/>
-  <link name="laser_link">
+  <!--_______________________ STEREO CAMERA _______________________-->
+  <link name="sensor_link">
     <collision>
-    <origin xyz="0 0 0" rpy="0 0 0"/>
-    <geometry>
-      <box size="${box_side} ${box_side} ${box_side}"/>
-    </geometry>
+      <origin xyz="0 0 0" rpy="0 0 0"/>
+      <geometry>
+        <box size="${box_side} ${box_side} ${box_side}"/>
+      </geometry>
     </collision>
     <visual>
-    <origin xyz="0 0 0" rpy="0 0 0"/>
-      <geometry>
-      <box size="${box_side} ${box_side} ${box_side}"/>
+      <origin xyz="0 0 0" rpy="0 0 0"/>
+      <geometry>
+        <box size="${box_side} ${box_side} ${box_side}"/>
       </geometry>
     </visual>
-    <inertial>
-      <mass value="1e-5" />
-      <origin xyz="0 0 0" rpy="0 0 0"/>
-      <inertia ixx="1e-6" ixy="0" ixz="0" iyy="1e-6" iyz="0" izz="1e-6" />
-    </inertial>
+    <xacro:sensor_inertial/>
   </link>
-  <joint name="laser_joint" type="fixed">
-    <axis xyz="0 0 1" />
-    <origin xyz="0 0 ${base_height + box_side/2}" rpy="0 0 0"/>
+  <!--_______________________ Stereocam Joint _______________________-->
+  <joint name="sensor_joint" type="fixed">
+    <origin xyz="0 0 ${wheel_dia+1}" rpy="0 0 0"/>
+    <axis xyz="1 0 0" rpy="0 0 0"/>
     <parent link="base_link"/>
-    <child link="laser_link"/>
+    <child link="sensor_link"/>
   </joint>
-<gazebo reference="laser_link">
-  <sensor type="ray" name="laser">
-    <pose>0 0 0 0 0 0</pose>
-    <visualize>true</visualize>
-    <update_rate>40</update_rate>
-    <ray>
-    <scan>
-    <horizontal>
-      <samples>720</samples>
-      <resolution>1</resolution>
-      <min_angle>-3.14159</min_angle>
-      <max_angle>3.14159</max_angle>
-    </horizontal>
-    </scan>
-    <range>
-    <min>0.10</min>
-    <max>30.0</max>
-    <resolution>0.01</resolution>
-    </range>
-    </ray>
-    <plugin name="gazebo_ros_head_hokuyo_controller" filename="libgazebo_ros_laser.so">
-      <topicName>/scan</topicName>
-      <frameName>laser_link</frameName>
-    </plugin>
-  </sensor>
-</gazebo>
-<link name="imu_link">
-  <inertial>
-    <mass value="0.001"/>
-    <origin rpy="0 0 0" xyz="0 0 0"/>
-    <inertia ixx="0.0001" ixy="0" ixz="0" iyy="0.000001" iyz="0" izz="0.0001"/>
-  </inertial>
-  <visual>
-    <origin rpy="0 0 0" xyz="0 0 0"/>
-    <geometry>
-      <box size="0.001 0.001 0.001"/>
-    </geometry>
-  </visual>
-  <collision>
-    <origin rpy="0 0 0" xyz="0 0 0"/>
-    <geometry>
-      <box size=".001 .001 .001"/>
-    </geometry>
-  </collision>
-</link>
-<joint name="imu_joint" type="fixed">
-  <axis xyz="1 0 0"/> <!-- 0 1 0 -->
-    <origin xyz="0 0 0"/>
-    <parent link="base_link"/>
-    <child link="imu_link"/>
-</joint>
-  <gazebo reference="imu_link">
-    <gravity>true</gravity>
-    <sensor name="imu_sensor" type="imu">
-      <always_on>true</always_on>
-      <update_rate>100</update_rate>
-      <visualize>true</visualize>
-      <topic>__default_topic__</topic>
-      <plugin filename="libgazebo_ros_imu_sensor.so" name="imu_plugin">
-        <topicName>imu_data</topicName>
-        <bodyName>imu_link</bodyName>
-        <updateRateHZ>10.0</updateRateHZ>
-        <gaussianNoise>0.0</gaussianNoise>
-        <xyzOffset>0 0 0</xyzOffset>
-        <rpyOffset>0 0 0</rpyOffset>
-        <frameName>imu_link</frameName>
-        <initialOrientationAsReference>false</initialOrientationAsReference>
-      </plugin>
-      <pose>0 0 0 0 0 0</pose>
-    </sensor>
-  </gazebo>
   <!-- SKID STEER PLUGIN -->
   <gazebo>
@@ -219,3 +146,59 @@
     </plugin>
   </gazebo>
+  <!-- Sensor plugin -->
+  <gazebo reference="sensor_link">
+    <sensor type="multicamera" name="stereo_camera">
+      <update_rate>30.0</update_rate>
+      <camera name="left">
+      <pose>${box_side} ${box_side/2} 0 0 0 0</pose>
+        <horizontal_fov>1.3962634</horizontal_fov>
+        <image>
+          <width>800</width>
+          <height>800</height>
+          <format>R8G8B8</format>
+        </image>
+        <clip>
+          <near>0.02</near>
+          <far>300</far>
+        </clip>
+        <noise>
+          <type>gaussian</type>
+          <mean>0.0</mean>
+          <stddev>0.007</stddev>
+        </noise>
+      </camera>
+      <camera name="right">
+        <pose>${box_side} -${box_side/2} 0 0 0 0</pose>
+        <horizontal_fov>1.3962634</horizontal_fov>
+        <image>
+          <width>800</width>
+          <height>800</height>
+          <format>R8G8B8</format>
+        </image>
+        <clip>
+          <near>0.02</near>
+          <far>300</far>
+        </clip>
+        <noise>
+          <type>gaussian</type>
+          <mean>0.0</mean>
+          <stddev>0.007</stddev>
+        </noise>
+      </camera>
+      <plugin name="stereo_camera_controller" filename="libgazebo_ros_multicamera.so">
+        <alwaysOn>true</alwaysOn>
+        <updateRate>30.0</updateRate>
+        <cameraName>stereo</cameraName>
+        <imageTopicName>image_raw</imageTopicName>
+        <cameraInfoTopicName>camera_info</cameraInfoTopicName>
+        <frameName>sensor_link</frameName>
+        <hackBaseline>0.07</hackBaseline>
+        <distortionK1>0.0</distortionK1>
+        <distortionK2>0.0</distortionK2>
+        <distortionK3>0.0</distortionK3>
+        <distortionT1>0.0</distortionT1>
+        <distortionT2>0.0</distortionT2>
+      </plugin>
+    </sensor>
+  </gazebo>
 </robot>

Commit message: Add mapping

File: src/wheelchair_description/urdf/wheelchair_body_stereo.xacro (robot description, xacro)
@@ -100,4 +100,26 @@
   <xacro:wheel left_right="left" rely="1"/>
   <xacro:wheel left_right="right" rely="-1"/>
+  <!-- LASER LINK -->
+  <link name="laser_link">
+    <collision>
+    <origin xyz="0 0 0" rpy="0 0 0"/>
+    <geometry>
+      <box size="${box_side} ${box_side} ${box_side}"/>
+    </geometry>
+    </collision>
+    <visual>
+    <origin xyz="0 0 0" rpy="0 0 0"/>
+      <geometry>
+      <box size="${box_side} ${box_side} ${box_side}"/>
+      </geometry>
+    </visual>
+    <xacro:sensor_inertial/>
+  </link>
+  <joint name="laser_joint" type="fixed">
+    <axis xyz="0 0 1" />
+    <origin xyz="0 0 ${base_height + box_side/2}" rpy="0 0 0"/>
+    <parent link="base_link"/>
+    <child link="laser_link"/>
+  </joint>
   <!--_______________________ STEREO CAMERA _______________________-->
   <link name="sensor_link">
@@ -132,10 +154,19 @@
       <wheelSeparation>0.5</wheelSeparation>
       <wheelDiameter>0.1</wheelDiameter>
-      <wheelAcceleration>1.0</wheelAcceleration>
-      <wheelTorque>5</wheelTorque>
+      <wheelAcceleration>0.5</wheelAcceleration>
+      <wheelTorque>50</wheelTorque>
       <robotBaseFrame>base_link</robotBaseFrame>
       <commandTopic>cmd_vel</commandTopic>
       <odometryTopic>odom</odometryTopic>
       <broadcastTF>false</broadcastTF>
+      <odometryFrame>odom</odometryFrame>
+      <odometrySource>world</odometrySource>
+      <publishOdomTF>true</publishOdomTF>
+      <robotBaseFrame>base_link</robotBaseFrame>
+      <publishWheelTF>false</publishWheelTF>
+      <publishTf>true</publishTf>
+      <publishWheelJointState>true</publishWheelJointState>
+      <legacyMode>false</legacyMode>
+      <rosDebugLevel>na</rosDebugLevel>
     </plugin>
   </gazebo>
@@ -146,5 +177,31 @@
     </plugin>
   </gazebo>
-  <!-- Sensor plugin -->
+    <!-- LASER PLUGIN -->
+  <gazebo reference="laser_link">
+    <sensor type="ray" name="laser">
+      <pose>0 0 0 0 0 0</pose>
+      <visualize>true</visualize>
+      <update_rate>40</update_rate>
+      <ray>
+      <scan>
+      <horizontal>
+        <samples>720</samples>
+        <resolution>1</resolution>
+        <min_angle>-3.14159</min_angle>
+        <max_angle>3.14159</max_angle>
+      </horizontal>
+      </scan>
+      <range>
+      <min>0.10</min>
+      <max>30.0</max>
+      <resolution>0.01</resolution>
+      </range>
+      </ray>
+      <plugin name="gazebo_ros_head_hokuyo_controller" filename="libgazebo_ros_laser.so">
+        <topicName>/scan</topicName>
+        <frameName>laser_link</frameName>
+      </plugin>
+    </sensor>
+  </gazebo>
   <gazebo reference="sensor_link">
     <sensor type="multicamera" name="stereo_camera">

Commit message: Spawn in environment with stereo image

File: src/wheelchair_description/urdf/wheelchair_body_stereo.xacro (robot description, xacro)
@@ -141,5 +141,5 @@
   <joint name="sensor_joint" type="fixed">
     <origin xyz="0 0 ${wheel_dia+1}" rpy="0 0 0"/>
-    <axis xyz="1 0 0" rpy="0 0 0"/>
+    <axis xyz="0 0 1" rpy="0 0 0"/>
     <parent link="base_link"/>
     <child link="sensor_link"/>
@@ -177,5 +177,5 @@
     </plugin>
   </gazebo>
-    <!-- LASER PLUGIN -->
+  <!-- LASER PLUGIN -->
   <gazebo reference="laser_link">
     <sensor type="ray" name="laser">
